Commit message: all gazebo spawn

File: robot_description/robot_description/urdf/robot_6dof_arm.xacro (robot description, xacro)
@@ -10,4 +10,61 @@
 <material name="Black"><color rgba="0.0 0.0 0.0 1.0"/></material>
 <material name="White"><color rgba="1.0 1.0 1.0 1.0"/></material>
+<!-- Example transmission (repeat for each joint) -->
+<transmission name="joint1_trans">
+  <type>transmission_interface/SimpleTransmission</type>
+  <actuator name="joint1_motor"/>
+  <joint name="base_link_link1"/>
+</transmission>
+<transmission name="joint2_trans">
+  <type>transmission_interface/SimpleTransmission</type>
+  <actuator name="joint2_motor"/>
+  <joint name="link1_link2"/>
+</transmission>
+<transmission name="joint3_trans">
+  <type>transmission_interface/SimpleTransmission</type>
+  <actuator name="joint3_motor"/>
+  <joint name="link2_link3"/>
+</transmission>
+<transmission name="joint4_trans">
+  <type>transmission_interface/SimpleTransmission</type>
+  <actuator name="joint4_motor"/>
+  <joint name="link3_link4"/>
+</transmission>
+<transmission name="joint5_trans">
+  <type>transmission_interface/SimpleTransmission</type>
+  <actuator name="joint5_motor"/>
+  <joint name="link4_link5"/>
+</transmission>
+<!--End effector-->
+<transmission name="joint6_trans">
+  <type>transmission_interface/SimpleTransmission</type>
+  <actuator name="joint6_motor"/>
+  <joint name="link5_tcp_connector"/>
+</transmission>
+<transmission name="joint7_trans">
+  <type>transmission_interface/SimpleTransmission</type>
+  <actuator name="joint7_motor"/>
+  <joint name="tcp_connector_gripper_right"/>
+</transmission>
+<transmission name="joint8_trans">
+  <type>transmission_interface/SimpleTransmission</type>
+  <actuator name="joint8_motor"/>
+  <joint name="tcp_connector_gripper_left"/>
+</transmission>
+<plugin name="ros2_control_node" filename="libros2_control_node.so">
+  <ros2_control>
+    <hardware>ros2_control_test_hardware/ActuatorHardware</hardware>
+    <joints>
+      <joint name="base_link_link1"/>
+      <joint name="link1_link2"/>
+      <joint name="link2_link3"/>
+      <joint name="link3_link4"/>
+      <joint name="link4_link5"/>
+      <joint name="link5_tcp_connector"/>
+      <joint name="tcp_connector_gripper_right"/>
+      <joint name="tcp_connector_gripper_left"/>
+    </joints>
+  </ros2_control>
+</plugin>
     <!-- Links -->
     <link name="base_link">
@@ -27,6 +84,7 @@
         <inertial>
             <origin xyz="0 0 0" rpy="0 0 0"/>
-            <mass value="1.0"/>
-            <inertia ixx="0.01" ixy="0.0" ixz="0.0" iyy="0.01" iyz="0.0" izz="0.01"/>
+            <mass value="5.0"/>
+            <!-- cylinder inertia (r=0.1, L=0.05) -->
+            <inertia ixx="0.013542" ixy="0.0" ixz="0.0" iyy="0.013542" iyz="0.0" izz="0.025000"/>
         </inertial>
     </link>
@@ -47,7 +105,8 @@
         <inertial>
             <origin xyz="0 0 0" rpy="0 0 0"/>
-            <mass value="1.0"/>
-            <inertia ixx="0.01" ixy="0.0" ixz="0.0" iyy="0.01" iyz="0.0" izz="0.01"/>
-            </inertial>
+            <mass value="2.0"/>
+            <!-- cylinder inertia (r=0.05, L=0.264) -->
+            <inertia ixx="0.012866" ixy="0.0" ixz="0.0" iyy="0.012866" iyz="0.0" izz="0.002500"/>
+        </inertial>
     </link>
     <joint name="base_link_link1" type="revolute">
@@ -74,6 +133,7 @@
         <inertial>
             <origin xyz="0 0 0" rpy="0 0 0"/>
-            <mass value="1.0"/>
-            <inertia ixx="0.01" ixy="0.0" ixz="0.0" iyy="0.01" iyz="0.0" izz="0.01"/>
+            <mass value="3.0"/>
+            <!-- cylinder inertia (r=0.05, L=0.85) -->
+            <inertia ixx="0.182500" ixy="0.0" ixz="0.0" iyy="0.182500" iyz="0.0" izz="0.003750"/>
         </inertial>
     </link>
@@ -101,6 +161,7 @@
         <inertial>
             <origin xyz="0 0 0" rpy="0 0 0"/>
-            <mass value="1.0"/>
-            <inertia ixx="0.01" ixy="0.0" ixz="0.0" iyy="0.01" iyz="0.0" izz="0.01"/>
+            <mass value="2.5"/>
+            <!-- cylinder inertia (r=0.05, L=0.68) -->
+            <inertia ixx="0.097896" ixy="0.0" ixz="0.0" iyy="0.097896" iyz="0.0" izz="0.003125"/>
         </inertial>
     </link>
@@ -128,6 +189,7 @@
         <inertial>
             <origin xyz="0 0 0" rpy="0 0 0"/>
-            <mass value="1.0"/>
-            <inertia ixx="0.01" ixy="0.0" ixz="0.0" iyy="0.01" iyz="0.0" izz="0.01"/>
+            <mass value="1.5"/>
+            <!-- cylinder inertia (r=0.05, L=0.13) -->
+            <inertia ixx="0.003050" ixy="0.0" ixz="0.0" iyy="0.003050" iyz="0.0" izz="0.001875"/>
         </inertial>
     </link>
@@ -156,5 +218,6 @@
             <origin xyz="0 0 0" rpy="0 0 0"/>
             <mass value="1.0"/>
-            <inertia ixx="0.01" ixy="0.0" ixz="0.0" iyy="0.01" iyz="0.0" izz="0.01"/>
+            <!-- cylinder inertia (r=0.05, L=0.17) -->
+            <inertia ixx="0.003033" ixy="0.0" ixz="0.0" iyy="0.003033" iyz="0.0" izz="0.001250"/>
         </inertial>
     </link>
@@ -183,6 +246,7 @@
         <inertial>
             <origin xyz="0 0 0" rpy="0 0 0"/>
-            <mass value="1.0"/>
-            <inertia ixx="0.01" ixy="0.0" ixz="0.0" iyy="0.01" iyz="0.0" izz="0.01"/>
+            <mass value="0.5"/>
+            <!-- box inertia (0.03 x 0.15 x 0.03) -->
+            <inertia ixx="0.000975" ixy="0.0" ixz="0.0" iyy="0.000075" iyz="0.0" izz="0.000975"/>
         </inertial>
     </link>
@@ -210,6 +274,7 @@
         <inertial>
             <origin xyz="0 0 0" rpy="0 0 0"/>
-            <mass value="1.0"/>
-            <inertia ixx="0.01" ixy="0.0" ixz="0.0" iyy="0.01" iyz="0.0" izz="0.01"/>
+            <mass value="0.2"/>
+            <!-- box inertia (0.01 x 0.01 x 0.1) -->
+            <inertia ixx="0.000168" ixy="0.0" ixz="0.0" iyy="0.000168" iyz="0.0" izz="0.000003"/>
         </inertial>
     </link>
@@ -237,6 +302,6 @@
         <inertial>
             <origin xyz="0 0 0" rpy="0 0 0"/>
-            <mass value="1.0"/>
-            <inertia ixx="0.01" ixy="0.0" ixz="0.0" iyy="0.01" iyz="0.0" izz="0.01"/>
+            <mass value="0.2"/>
+            <inertia ixx="0.000168" ixy="0.0" ixz="0.0" iyy="0.000168" iyz="0.0" izz="0.000003"/>
         </inertial>
     </link>
@@ -248,3 +313,8 @@
         <limit lower="0.0" upper="0.055" effort="0.5" velocity="1000.0"/>
     </joint>
+    <link name="world"/>
+    <joint name="fixed_base_joint" type="fixed">
+        <parent link="world"/>
+        <child link="base_link"/>
+    </joint>
 </robot>

File: robot_description/robot_description/urdf/test.xacro (robot description, xacro)
@@ -1,4 +1,70 @@
-<?xml version="1.0"?>
-<robot name="robot_6dof">
+<!-- <?xml version="1.0"?>
+<robot xmlns:xacro="http://www.ros.org/wiki/xacro" name="robot_6dof_arm">
+<material name="Grey"><color rgba="0.5 0.5 0.5 1.0"/></material>
+<material name="Blue"><color rgba="0.0 0.0 1.0 1.0"/></material>
+<material name="Green"><color rgba="0.0 1.0 0.0 1.0"/></material>
+<material name="Red"><color rgba="1.0 0.0 0.0 1.0"/></material>
+<material name="Yellow"><color rgba="1.0 1.0 0.0 1.0"/></material>
+<material name="Cyan"><color rgba="0.0 1.0 1.0 1.0"/></material>
+<material name="Magenta"><color rgba="1.0 0.0 1.0 1.0"/></material>
+<material name="Black"><color rgba="0.0 0.0 0.0 1.0"/></material>
+<material name="White"><color rgba="1.0 1.0 1.0 1.0"/></material>
+<!-- Example transmission (repeat for each joint) -->
+<transmission name="joint1_trans">
+  <type>transmission_interface/SimpleTransmission</type>
+  <actuator name="joint1_motor"/>
+  <joint name="base_link_link1"/>
+</transmission>
+<transmission name="joint2_trans">
+  <type>transmission_interface/SimpleTransmission</type>
+  <actuator name="joint2_motor"/>
+  <joint name="link1_link2"/>
+</transmission>
+<transmission name="joint3_trans">
+  <type>transmission_interface/SimpleTransmission</type>
+  <actuator name="joint3_motor"/>
+  <joint name="link2_link3"/>
+</transmission>
+<transmission name="joint4_trans">
+  <type>transmission_interface/SimpleTransmission</type>
+  <actuator name="joint4_motor"/>
+  <joint name="link3_link4"/>
+</transmission>
+<transmission name="joint5_trans">
+  <type>transmission_interface/SimpleTransmission</type>
+  <actuator name="joint5_motor"/>
+  <joint name="link4_link5"/>
+</transmission>
+<!--End effector-->
+<transmission name="joint6_trans">
+  <type>transmission_interface/SimpleTransmission</type>
+  <actuator name="joint6_motor"/>
+  <joint name="link5_tcp_connector"/>
+</transmission>
+<transmission name="joint7_trans">
+  <type>transmission_interface/SimpleTransmission</type>
+  <actuator name="joint7_motor"/>
+  <joint name="tcp_connector_gripper_right"/>
+</transmission>
+<transmission name="joint8_trans">
+  <type>transmission_interface/SimpleTransmission</type>
+  <actuator name="joint8_motor"/>
+  <joint name="tcp_connector_gripper_left"/>
+</transmission>
+<plugin name="ros2_control_node" filename="libros2_control_node.so">
+  <ros2_control>
+    <hardware>ros2_control_test_hardware/ActuatorHardware</hardware>
+    <joints>
+      <joint name="base_link_link1"/>
+      <joint name="link1_link2"/>
+      <joint name="link2_link3"/>
+      <joint name="link3_link4"/>
+      <joint name="link4_link5"/>
+      <joint name="link5_tcp_connector"/>
+      <joint name="tcp_connector_gripper_right"/>
+      <joint name="tcp_connector_gripper_left"/>
+    </joints>
+  </ros2_control>
+</plugin>
     <!-- Links -->
     <link name="base_link">
@@ -239,117 +305,244 @@
         <limit lower="0.0" upper="0.055" effort="0.5" velocity="1000.0"/>
     </joint>
-</robot>
-<?xml version="1.0"?>
-<robot xmlns:xacro="http://www.ros.org/wiki/xacro" name="my_6dof_arm">
-  <!-- Macro to create a simple box link -->
-  <xacro:macro name="simple_link" params="name xyz rpy size color">
-    <link name="${name}">
-      <visual>
-        <origin xyz="${xyz}" rpy="${rpy}"/>
-        <geometry>
-          <box size="${size}"/>
-        </geometry>
-        <material name="${color}"/>
-      </visual>
-      <collision>
-        <origin xyz="${xyz}" rpy="${rpy}"/>
-        <geometry>
-          <box size="${size}"/>
-        </geometry>
-      </collision>
-      <inertial>
-        <origin xyz="0 0 0" rpy="0 0 0"/>
-        <mass value="1.0"/>
-        <inertia ixx="0.01" ixy="0.0" ixz="0.0" iyy="0.01" iyz="0.0" izz="0.01"/>
-      </inertial>
-    </link>
-  </xacro:macro>
-  <!-- Links -->
-  <xacro:simple_link name="base_link" xyz="0 0 0.05" rpy="0 0 0" size="0.1 0.1 0.1" color="Grey"/>
-  <xacro:simple_link name="link_1" xyz="0 0 0.1" rpy="0 0 0" size="0.05 0.05 0.2" color="Blue"/>
-  <xacro:simple_link name="link_2" xyz="0 0 0.2" rpy="0 0 0" size="0.05 0.05 0.2" color="Green"/>
-  <xacro:simple_link name="link_3" xyz="0 0 0.2" rpy="0 0 0" size="0.05 0.05 0.2" color="Red"/>
-  <xacro:simple_link name="link_4" xyz="0 0 0.15" rpy="0 0 0" size="0.04 0.04 0.15" color="Yellow"/>
-  <xacro:simple_link name="link_5" xyz="0 0 0.1" rpy="0 0 0" size="0.03 0.03 0.1" color="Cyan"/>
-  <xacro:simple_link name="link_6" xyz="0 0 0.1" rpy="0 0 0" size="0.02 0.02 0.1" color="Magenta"/>
-  <xacro:simple_link name="ee_link" xyz="0 0 0.05" rpy="0 0 0" size="0.05 0.05 0.05" color="White"/>
-  <!-- Joints (same as before) -->
-  <joint name="joint_1" type="revolute">
-    <parent link="base_link"/>
-    <child link="link_1"/>
-    <origin xyz="0 0 0.1" rpy="0 0 0"/>
-    <axis xyz="0 0 1"/>
-    <limit lower="-3.14" upper="3.14" effort="50" velocity="1.0"/>
-  </joint>
-  <joint name="joint_2" type="revolute">
-    <parent link="link_1"/>
-    <child link="link_2"/>
-    <origin xyz="0 0 0.2" rpy="0 0 0"/>
-    <axis xyz="0 1 0"/>
-    <limit lower="-3.14" upper="3.14" effort="50" velocity="1.0"/>
-  </joint>
-  <joint name="joint_3" type="revolute">
-    <parent link="link_2"/>
-    <child link="link_3"/>
-    <origin xyz="0 0 0.2" rpy="0 0 0"/>
-    <axis xyz="0 1 0"/>
-    <limit lower="-3.14" upper="3.14" effort="50" velocity="1.0"/>
-  </joint>
-  <joint name="joint_4" type="revolute">
-    <parent link="link_3"/>
-    <child link="link_4"/>
-    <origin xyz="0 0 0.15" rpy="0 0 0"/>
-    <axis xyz="1 0 0"/>
-    <limit lower="-3.14" upper="3.14" effort="50" velocity="1.0"/>
-  </joint>
-  <joint name="joint_5" type="revolute">
-    <parent link="link_4"/>
-    <child link="link_5"/>
-    <origin xyz="0 0 0.1" rpy="0 0 0"/>
-    <axis xyz="0 1 0"/>
-    <limit lower="-3.14" upper="3.14" effort="50" velocity="1.0"/>
-  </joint>
-  <joint name="joint_6" type="revolute">
-    <parent link="link_5"/>
-    <child link="link_6"/>
-    <origin xyz="0 0 0.1" rpy="0 0 0"/>
-    <axis xyz="1 0 0"/>
-    <limit lower="-3.14" upper="3.14" effort="50" velocity="1.0"/>
-  </joint>
-  <joint name="ee_joint" type="fixed">
-    <parent link="link_6"/>
-    <child link="ee_link"/>
-    <origin xyz="0 0 0.05" rpy="0 0 0"/>
-  </joint>
-  <!-- ros2_control transmissions (same as before) -->
-  <transmission name="joint_1_trans">
-    <type>transmission_interface/SimpleTransmission</type>
-    <joint name="joint_1"/>
-    <actuator name="joint_1_motor"/>
-  </transmission>
-  <transmission name="joint_2_trans">
-    <type>transmission_interface/SimpleTransmission</type>
-    <joint name="joint_2"/>
-    <actuator name="joint_2_motor"/>
-  </transmission>
-  <transmission name="joint_3_trans">
-    <type>transmission_interface/SimpleTransmission</type>
-    <joint name="joint_3"/>
-    <actuator name="joint_3_motor"/>
-  </transmission>
-  <transmission name="joint_4_trans">
-    <type>transmission_interface/SimpleTransmission</type>
-    <joint name="joint_4"/>
-    <actuator name="joint_4_motor"/>
-  </transmission>
-  <transmission name="joint_5_trans">
-    <type>transmission_interface/SimpleTransmission</type>
-    <joint name="joint_5"/>
-    <actuator name="joint_5_motor"/>
-  </transmission>
-  <transmission name="joint_6_trans">
-    <type>transmission_interface/SimpleTransmission</type>
-    <joint name="joint_6"/>
-    <actuator name="joint_6_motor"/>
-  </transmission>
-</robot>
+</robot> -->
+<!-- <?xml version="1.0"?>
+<robot name="robot_6dof">
+    <!-- Links -->
+    <link name="base_link">
+        <visual>
+            <origin xyz="0.0 0.0 0.025" rpy="0.0 0.0 0.0"/>
+            <geometry>
+                <cylinder radius="0.1" length="0.05"/>
+            </geometry>
+            <material name="Grey"/>
+        </visual>
+        <collision>
+            <origin xyz="0.0 0.0 0.025" rpy="0.0 0.0 0.0"/>
+            <geometry>
+                <cylinder radius="0.1" length="0.05"/>
+            </geometry>
+        </collision>
+        <inertial>
+            <origin xyz="0 0 0" rpy="0 0 0"/>
+            <mass value="1.0"/>
+            <inertia ixx="0.01" ixy="0.0" ixz="0.0" iyy="0.01" iyz="0.0" izz="0.01"/>
+        </inertial>
+    </link>
+    <link name="link_1">
+        <visual>
+            <origin xyz="0.0 0.0 0.132" rpy="0.0 0.0 0.0"/>
+            <geometry>
+                <cylinder radius="0.05" length="0.264"/>
+            </geometry>
+            <material name="Blue"/>
+        </visual>
+        <collision>
+            <origin xyz="0.0 0.0 0.132" rpy="0.0 0.0 0.0"/>
+            <geometry>
+                <cylinder radius="0.05" length="0.264"/>
+            </geometry>
+        </collision>
+        <inertial>
+            <origin xyz="0 0 0" rpy="0 0 0"/>
+            <mass value="1.0"/>
+            <inertia ixx="0.01" ixy="0.0" ixz="0.0" iyy="0.01" iyz="0.0" izz="0.01"/>
+            </inertial>
+    </link>
+    <joint name="base_link_link1" type="revolute">
+        <parent link="base_link"/>
+        <child link="link_1"/>
+        <origin xyz="0.0 0.0 0.05" rpy="0 0 0"/>
+        <axis xyz="0 0 1"/>
+        <limit lower="-3.14159" upper="3.14159" effort="0.5" velocity="1000.0"/>
+    </joint>
+    <link name="link_2">
+        <visual>
+            <origin xyz="0.0 0.0 0.425" rpy="0.0 0.0 0.0"/>
+            <geometry>
+                <cylinder radius="0.05" length="0.850"/>
+            </geometry>
+            <material name="Green"/>
+        </visual>
+        <collision>
+            <origin xyz="0.0 0.0 0.425" rpy="0.0 0.0 0.0"/>
+            <geometry>
+                <cylinder radius="0.05" length="0.850"/>
+            </geometry>
+        </collision>
+        <inertial>
+            <origin xyz="0 0 0" rpy="0 0 0"/>
+            <mass value="1.0"/>
+            <inertia ixx="0.01" ixy="0.0" ixz="0.0" iyy="0.01" iyz="0.0" izz="0.01"/>
+        </inertial>
+    </link>
+    <joint name="link1_link2" type="revolute">
+        <parent link="link_1"/>
+        <child link="link_2"/>
+        <origin xyz="0.0 0.1 0.214" rpy="0 0 0"/>
+        <axis xyz="0 1 0"/>
+        <limit lower="-2.50" upper="2.50" effort="0.5" velocity="1000.0"/>
+    </joint>
+    <link name="link_3">
+        <visual>
+            <origin xyz="0.0 0.0 0.340" rpy="0.0 0.0 0.0"/>
+            <geometry>
+                <cylinder radius="0.05" length="0.680"/>
+            </geometry>
+            <material name="Red"/>
+        </visual>
+        <collision>
+            <origin xyz="0.0 0.0 0.340" rpy="0.0 0.0 0.0"/>
+            <geometry>
+                <cylinder radius="0.05" length="0.680"/>
+            </geometry>
+        </collision>
+        <inertial>
+            <origin xyz="0 0 0" rpy="0 0 0"/>
+            <mass value="1.0"/>
+            <inertia ixx="0.01" ixy="0.0" ixz="0.0" iyy="0.01" iyz="0.0" izz="0.01"/>
+        </inertial>
+    </link>
+    <joint name="link2_link3" type="revolute">
+        <parent link="link_2"/>
+        <child link="link_3"/>
+        <origin xyz="0.0 -0.1 0.8" rpy="0 0 0"/>
+        <axis xyz="0 1 0"/>
+        <limit lower="-3.14" upper="3.14" effort="0.5" velocity="1000.0"/>
+    </joint>
+    <link name="link_4">
+        <visual>
+            <origin xyz="0.0 0.0 0.065" rpy="0.0 0.0 0.0"/>
+            <geometry>
+                <cylinder radius="0.05" length="0.130"/>
+            </geometry>
+            <material name="Yellow"/>
+        </visual>
+        <collision>
+            <origin xyz="0.0 0.0 0.065" rpy="0.0 0.0 0.0"/>
+            <geometry>
+                <cylinder radius="0.05" length="0.130"/>
+            </geometry>
+        </collision>
+        <inertial>
+            <origin xyz="0 0 0" rpy="0 0 0"/>
+            <mass value="1.0"/>
+            <inertia ixx="0.01" ixy="0.0" ixz="0.0" iyy="0.01" iyz="0.0" izz="0.01"/>
+        </inertial>
+    </link>
+    <joint name="link3_link4" type="revolute">
+        <parent link="link_3"/>
+        <child link="link_4"/>
+        <origin xyz="0.0 0.1 0.630" rpy="0 0 0"/>
+        <axis xyz="0 1 0"/>
+        <limit lower="-3.14" upper="3.14" effort="0.5" velocity="1000.0"/>
+    </joint>
+    <link name="link_5">
+        <visual>
+            <origin xyz="0.0 0.0 0.035" rpy="0.0 0.0 0.0"/>
+            <geometry>
+                <cylinder radius="0.05" length="0.170"/>
+            </geometry>
+            <material name="Cyan"/>
+        </visual>
+        <collision>
+            <origin xyz="0.0 0.0 0.035" rpy="0.0 0.0 0.0"/>
+            <geometry>
+                <cylinder radius="0.05" length="0.170"/>
+            </geometry>
+        </collision>
+        <inertial>
+            <origin xyz="0 0 0" rpy="0 0 0"/>
+            <mass value="1.0"/>
+            <inertia ixx="0.01" ixy="0.0" ixz="0.0" iyy="0.01" iyz="0.0" izz="0.01"/>
+        </inertial>
+    </link>
+    <joint name="link4_link5" type="revolute">
+        <parent link="link_4"/>
+        <child link="link_5"/>
+        <origin xyz="0.0 0.0 0.180" rpy="0 1.57 0"/>
+        <axis xyz="1 0 0"/>
+        <limit lower="-3.14" upper="3.14" effort="0.5" velocity="1000.0"/>
+    </joint>
+    <!--build the TCP or end effector-->
+    <link name="tcp_connector">
+        <visual>
+            <origin xyz="0.0 0.0 0.0125" rpy="0.0 0.0 0.0"/>
+            <geometry>
+                <box size="0.03 0.150 0.03"/>
+            </geometry>
+            <material name="White"/>
+        </visual>
+        <collision>
+            <origin xyz="0.0 0.0 0.0125" rpy="0.0 0.0 0.0"/>
+            <geometry>
+                <box size="0.03 0.150 0.03"/>
+            </geometry>
+        </collision>
+        <inertial>
+            <origin xyz="0 0 0" rpy="0 0 0"/>
+            <mass value="1.0"/>
+            <inertia ixx="0.01" ixy="0.0" ixz="0.0" iyy="0.01" iyz="0.0" izz="0.01"/>
+        </inertial>
+    </link>
+    <joint name="link5_tcp_connector" type="revolute">
+        <parent link="link_5"/>
+        <child link="tcp_connector"/>
+        <origin xyz="0.0 0.0 0.120" rpy="0 0 0"/>
+        <axis xyz="0 0 1"/>
+        <limit lower="-3.14" upper="3.14" effort="0.5" velocity="1000.0"/>
+    </joint>
+    <link name="gripper_right">
+        <visual>
+            <origin xyz="0.0 0.0 0.05" rpy="0.0 0.0 0.0"/>
+            <geometry>
+                <box size="0.01 0.01 0.1"/>
+            </geometry>
+            <material name="Black"/>
+        </visual>
+        <collision>
+            <origin xyz="0.0 0.0 0.05" rpy="0.0 0.0 0.0"/>
+            <geometry>
+                <box size="0.01 0.01 0.1"/>
+            </geometry>
+        </collision>
+        <inertial>
+            <origin xyz="0 0 0" rpy="0 0 0"/>
+            <mass value="1.0"/>
+            <inertia ixx="0.01" ixy="0.0" ixz="0.0" iyy="0.01" iyz="0.0" izz="0.01"/>
+        </inertial>
+    </link>
+    <joint name="tcp_connector_gripper_right" type="prismatic">
+        <parent link="tcp_connector"/>
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