Commit message: Feat: Camera spawn in gazebo

File: robot_description/robot_description/urdf/overhead_camera.xacro (robot description, xacro)
@@ -7,13 +7,11 @@
         roll='0.0' pitch='-1.5708' yaw='0.0'
         fov='1.0472' width='1280' height='720' update_rate='30'
-        topic='/overhead_cam' ">
-    <!-- Base link attached to world -->
+        topic='/overhead_camera/image_raw' ">
     <link name="${prefix}_base_link"/>
     <joint name="${prefix}_fixed_joint" type="fixed">
-      <parent link="world"/>
+      <parent link="tcp_connector"/>
       <child  link="${prefix}_base_link"/>
       <origin xyz="${x} ${y} ${z}" rpy="${roll} ${pitch} ${yaw}"/>
     </joint>
-    <!-- Camera link -->
     <link name="${prefix}_camera_link"/>
     <joint name="${prefix}_camera_joint" type="fixed">
@@ -22,7 +20,11 @@
       <origin xyz="0 0 0" rpy="0 0 0"/>
     </joint>
-    <!-- Gazebo camera sensor -->
+    <gazebo>
+      <plugin name='gz::sim::systems::Sensors' filename='gz-sim-sensors-system'>
+          <render_engine>ogre2</render_engine>
+      </plugin>
+    </gazebo>
     <gazebo reference="${prefix}_camera_link">
-      <sensor name="${prefix}_camera_sensor" type="camera">
+      <sensor name="${prefix}_camera" type="camera">
         <pose>0 0 0 0 0 0</pose>
         <camera>
@@ -37,8 +39,11 @@
             <far>10</far>
           </clip>
+          <optical_frame_id>${prefix}_camera_link</optical_frame_id>
+          <camera_info_topic>/overhead_camera/camera_info</camera_info_topic>
         </camera>
-        <always_on>true</always_on>
+        <always_on>1</always_on>
         <update_rate>${update_rate}</update_rate>
         <visualize>true</visualize>
+        <topic>${topic}</topic>
       </sensor>
     </gazebo>

File: robot_description/robot_description/urdf/robot_6dof_arm.urdf.xacro (robot description, xacro)
@@ -1,16 +1,16 @@
 <?xml version="1.0"?>
 <robot xmlns:xacro="http://www.ros.org/wiki/xacro" name="robot_6dof_arm">
-<xacro:include filename="$(find robot_description)/urdf/overhead_camera.xacro"/>
-<!-- Instantiate the overhead camera macro -->
-<xacro:overhead_camera
-prefix="overhead"
-x="0.0"
-y="0.0"
-z="1.5"
-roll="0.0"
-pitch="-1.5708"
-yaw="0.0"
-topic="/overhead_camera/image_raw"
-/>
+    <xacro:include filename="overhead_camera.xacro"/>
+    <xacro:overhead_camera
+        prefix="overhead"
+        x="0.0"
+        y="0.0"
+        z="1.5"
+        roll="0.0"
+        pitch="-1.5708"
+        yaw="0.0"
+        topic="/overhead_camera/image_raw"
+    />
+    <link name="world"/>
     <material name="Grey"><color rgba="0.5 0.5 0.5 1.0"/></material>
     <material name="Blue"><color rgba="0.0 0.0 1.0 1.0"/></material>
@@ -22,5 +22,4 @@
     <material name="Black"><color rgba="0.0 0.0 0.0 1.0"/></material>
     <material name="White"><color rgba="1.0 1.0 1.0 1.0"/></material>
-    <!-- Example transmission (repeat for each joint) -->
     <transmission name="joint1_trans">
     <type>transmission_interface/SimpleTransmission</type>
@@ -48,5 +47,4 @@
     <joint name="link4_link5"/>
     </transmission>
-    <!--End effector-->
     <transmission name="joint6_trans">
     <type>transmission_interface/SimpleTransmission</type>
@@ -65,13 +63,12 @@
     </transmission>
     <gazebo>
-        <initial_position xyz="0 0 0"/>
-        <plugin filename="gz_ros2_control-system"
-                name="gz_ros2_control::GazeboSimROS2ControlPlugin">
-            <parameters>$(find robot_description)/config/controllers.yaml</parameters>
+        <plugin filename="ign_ros2_control-system"
+                name="ign_ros2_control::IgnitionROS2ControlPlugin">
+            <parameters>$(find robot_description)/robot_description/config/controllers.yaml</parameters>
         </plugin>
     </gazebo>
     <ros2_control name="IgnitionSystem" type="system">
         <hardware>
-            <plugin>gz_ros2_control/GazeboSimSystem</plugin>
+            <plugin>ign_ros2_control/IgnitionSystem</plugin>
         </hardware>
         <joint name="base_link_link1">
@@ -104,5 +101,5 @@
                 <param name="min">-1.57</param>
                 <param name="max">1.57</param>
-            </command_interface>
+             </command_interface>
             <state_interface name="position"/>
             <state_interface name="velocity"/>
@@ -132,5 +129,5 @@
             <state_interface name="velocity"/>
         </joint>
-        <joint name="tcp_connector_gripper_left">
+         <joint name="tcp_connector_gripper_left">
             <command_interface name="position">
                 <param name="min">-0.055</param>
@@ -141,5 +138,4 @@
         </joint>
     </ros2_control>
-    <!-- Links -->
     <link name="base_link">
         <visual>
@@ -148,5 +144,5 @@
                 <cylinder radius="0.1" length="0.05"/>
             </geometry>
-            <material name="Grey"/>
+             <material name="Grey"/>
         </visual>
         <collision>
@@ -157,7 +153,6 @@
         </collision>
         <inertial>
-            <origin xyz="0 0 0" rpy="0 0 0"/>
+             <origin xyz="0 0 0" rpy="0 0 0"/>
             <mass value="5.0"/>
-            <!-- cylinder inertia (r=0.1, L=0.05) -->
             <inertia ixx="0.013542" ixy="0.0" ixz="0.0" iyy="0.013542" iyz="0.0" izz="0.025000"/>
         </inertial>
@@ -173,5 +168,5 @@
         <collision>
             <origin xyz="0.0 0.0 0.132" rpy="0.0 0.0 0.0"/>
-            <geometry>
+             <geometry>
                 <cylinder radius="0.05" length="0.264"/>
             </geometry>
@@ -180,5 +175,4 @@
             <origin xyz="0 0 0" rpy="0 0 0"/>
             <mass value="2.0"/>
-            <!-- cylinder inertia (r=0.05, L=0.264) -->
             <inertia ixx="0.012866" ixy="0.0" ixz="0.0" iyy="0.012866" iyz="0.0" izz="0.002500"/>
         </inertial>
@@ -200,5 +194,5 @@
         </visual>
         <collision>
-            <origin xyz="0.0 0.0 0.425" rpy="0.0 0.0 0.0"/>
+           <origin xyz="0.0 0.0 0.425" rpy="0.0 0.0 0.0"/>
             <geometry>
                 <cylinder radius="0.05" length="0.850"/>
@@ -207,6 +201,5 @@
         <inertial>
             <origin xyz="0 0 0" rpy="0 0 0"/>
-            <mass value="3.0"/>
-            <!-- cylinder inertia (r=0.05, L=0.85) -->
+             <mass value="3.0"/>
             <inertia ixx="0.182500" ixy="0.0" ixz="0.0" iyy="0.182500" iyz="0.0" izz="0.003750"/>
         </inertial>
@@ -225,5 +218,5 @@
                 <cylinder radius="0.05" length="0.680"/>
             </geometry>
-            <material name="Red"/>
+             <material name="Red"/>
         </visual>
         <collision>
@@ -234,7 +227,6 @@
         </collision>
         <inertial>
-            <origin xyz="0 0 0" rpy="0 0 0"/>
+           <origin xyz="0 0 0" rpy="0 0 0"/>
             <mass value="2.5"/>
-            <!-- cylinder inertia (r=0.05, L=0.68) -->
             <inertia ixx="0.097896" ixy="0.0" ixz="0.0" iyy="0.097896" iyz="0.0" izz="0.003125"/>
         </inertial>
@@ -251,22 +243,21 @@
             <origin xyz="0.0 0.0 0.065" rpy="0.0 0.0 0.0"/>
             <geometry>
+                 <cylinder radius="0.05" length="0.130"/>
+            </geometry>
+            <material name="Yellow"/>
+        </visual>
+        <collision>
+            <origin xyz="0.0 0.0 0.065" rpy="0.0 0.0 0.0"/>
+            <geometry>
                 <cylinder radius="0.05" length="0.130"/>
-            </geometry>
-            <material name="Yellow"/>
-        </visual>
-        <collision>
-            <origin xyz="0.0 0.0 0.065" rpy="0.0 0.0 0.0"/>
-            <geometry>
-                <cylinder radius="0.05" length="0.130"/>
-            </geometry>
+             </geometry>
         </collision>
         <inertial>
             <origin xyz="0 0 0" rpy="0 0 0"/>
             <mass value="1.5"/>
-            <!-- cylinder inertia (r=0.05, L=0.13) -->
             <inertia ixx="0.003050" ixy="0.0" ixz="0.0" iyy="0.003050" iyz="0.0" izz="0.001875"/>
         </inertial>
     </link>
-    <joint name="link3_link4" type="revolute">
+     <joint name="link3_link4" type="revolute">
         <parent link="link_3"/>
         <child link="link_4"/>
@@ -278,5 +269,5 @@
         <visual>
             <origin xyz="0.0 0.0 0.035" rpy="0.0 0.0 0.0"/>
-            <geometry>
+             <geometry>
                 <cylinder radius="0.05" length="0.170"/>
             </geometry>
@@ -286,5 +277,5 @@
             <origin xyz="0.0 0.0 0.035" rpy="0.0 0.0 0.0"/>
             <geometry>
-                <cylinder radius="0.05" length="0.170"/>
+                 <cylinder radius="0.05" length="0.170"/>
             </geometry>
         </collision>
@@ -292,5 +283,4 @@
             <origin xyz="0 0 0" rpy="0 0 0"/>
             <mass value="1.0"/>
-            <!-- cylinder inertia (r=0.05, L=0.17) -->
             <inertia ixx="0.003033" ixy="0.0" ixz="0.0" iyy="0.003033" iyz="0.0" izz="0.001250"/>
         </inertial>
@@ -303,7 +293,6 @@
         <limit lower="-3.14" upper="3.14" effort="50.0" velocity="1000.0"/>
     </joint>
-    <!--build the TCP or end effector-->
     <link name="tcp_connector">
-        <visual>
+       <visual>
             <origin xyz="0.0 0.0 0.0125" rpy="0.0 0.0 0.0"/>
             <geometry>
@@ -313,5 +302,5 @@
         </visual>
         <collision>
-            <origin xyz="0.0 0.0 0.0125" rpy="0.0 0.0 0.0"/>
+             <origin xyz="0.0 0.0 0.0125" rpy="0.0 0.0 0.0"/>
             <geometry>
                 <box size="0.03 0.150 0.03"/>
@@ -320,6 +309,5 @@
         <inertial>
             <origin xyz="0 0 0" rpy="0 0 0"/>
-            <mass value="0.5"/>
-            <!-- box inertia (0.03 x 0.15 x 0.03) -->
+             <mass value="0.5"/>
             <inertia ixx="0.000975" ixy="0.0" ixz="0.0" iyy="0.000075" iyz="0.0" izz="0.000975"/>
         </inertial>
@@ -338,5 +326,5 @@
                 <box size="0.01 0.01 0.1"/>
             </geometry>
-            <material name="Black"/>
+             <material name="Black"/>
         </visual>
         <collision>
@@ -347,7 +335,6 @@
         </collision>
         <inertial>
-            <origin xyz="0 0 0" rpy="0 0 0"/>
+           <origin xyz="0 0 0" rpy="0 0 0"/>
             <mass value="0.2"/>
-            <!-- box inertia (0.01 x 0.01 x 0.1) -->
             <inertia ixx="0.000168" ixy="0.0" ixz="0.0" iyy="0.000168" iyz="0.0" izz="0.000003"/>
         </inertial>
@@ -355,5 +342,5 @@
     <joint name="tcp_connector_gripper_right" type="prismatic">
         <parent link="tcp_connector"/>
-        <child link="gripper_right"/>
+         <child link="gripper_right"/>
         <origin xyz="0.0 -0.065 0.03" rpy="0 0 0"/>
         <axis xyz="0 1 0"/>
@@ -364,13 +351,13 @@
             <origin xyz="0.0 0.0 0.05" rpy="0.0 0.0 0.0"/>
             <geometry>
+                 <box size="0.01 0.01 0.1"/>
+            </geometry>
+            <material name="Black"/>
+        </visual>
+        <collision>
+            <origin xyz="0.0 0.0 0.05" rpy="0.0 0.0 0.0"/>
+            <geometry>
                 <box size="0.01 0.01 0.1"/>
-            </geometry>
-            <material name="Black"/>
-        </visual>
-        <collision>
-            <origin xyz="0.0 0.0 0.05" rpy="0.0 0.0 0.0"/>
-            <geometry>
-                <box size="0.01 0.01 0.1"/>
-            </geometry>
+             </geometry>
         </collision>
         <inertial>
@@ -387,5 +374,4 @@
         <limit lower="-0.055" upper="0.0" effort="50.0" velocity="1000.0"/>
     </joint>
-    <link name="world"/>
     <joint name="fixed_base_joint" type="fixed">
         <parent link="world"/>
